File: hardware/energy-monitor.kicad_pcb (KiCad board)
At the start: 2 copper layers, 40 x 40 mm, 40 parts, among them P1 CON-SENSOR2, P3 BOOT, P4 DEBUG, U1 XMC110024, U2 TLV272IS, U3 DRILL, U4 DRILL, U5 DRILL, U6 DRILL, U7 phone-jack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

Commit message: changed processor to XMC1300
Parts:
- U1: value XMC110024 -> XMC1300
Changed lines of the file:
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@@
-(kicad_pcb (version 20171130) (host pcbnew 5.0.2-bee76a0~70~ubuntu18.04.1)
+(kicad_pcb (version 20171130) (host pcbnew 5.0.2-bee76a0~70~ubuntu18.10.1)
   (general
     (thickness 1.6)
@@
       (effects (font (size 0.3 0.3) (thickness 0.075)))
     )
-    (fp_text value XMC110024 (at 0 0.8) (layer F.Fab)
+    (fp_text value XMC1300 (at 0 0.8) (layer F.Fab)
       (effects (font (size 0.3 0.3) (thickness 0.075)))
     )
